File: Hardware/MyoWare_Cable_Shield.brd (EAGLE design)
At the start: 52.1 x 20.7 mm, 18 parts

Commit message: Removed RoHS claim
Parts:
- removed U$3: (no value), SparkFun-Aesthetics:ROHS_LOGO_0.18_IN
- removed U$5: (no value), SparkFun-Aesthetics:NO_PB_LOGO_0.120
Changed lines of the file:
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@@
 </autorouter>
 <elements>
-<element name="U$5" library="SparkFun-Aesthetics" package="NO_PB_LOGO_0.120" value="" x="14.40815" y="-1.905" rot="MR0"/>
 <element name="U$6" library="advancer-technologies" package="ADVANCER_LOGO" value="" x="-13.08735" y="7.2263"/>
-<element name="U$3" library="SparkFun-Aesthetics" package="ROHS_LOGO_0.18_IN" value="" x="-9.55675" y="-1.8415" smashed="yes" rot="MR0"/>
 <element name="JP6" library="SparkFun-Connectors" package="1X03_NO_SILK" value="Power" x="22.0345" y="2.54" smashed="yes" rot="R270"/>
 <element name="LOGO" library="advancer-technologies" package="MYOWARE_LOGO" value="" x="0" y="-0.889"/>
